Commit message: [update] tuned footprint

File: junbot/junbot_description/urdf/turtlebot3_jun.urdf.xacro (robot description, xacro)
@@ -141,5 +141,5 @@
     <parent link="base_link"/>
     <child link="laser"/>
-    <origin xyz="0.3 0 0.02" rpy="0 0 0"/>
+    <origin xyz="0.25 -0.01 0.02" rpy="0 0 0"/>
   </joint>
   <link name="laser">
